File: Edgeberry_console_cartridge.kicad_pcb (KiCad board)
At the start: 2 copper layers, 49.8 x 63.2 mm, 88 parts, among them J1 USB_B, J3 Screw_Terminal_01x03, U1 FT232RL, U2 MCP2515, U3 MCP2562, Y1 16MHz

Commit message: cleanup
Other:
- board text added: "Console & CAN, Rev. 1.5, mid 2024"
- board text added: "EDGEBERRY HARDWARE CARTRIDGE"
- board text removed: "Console & CAN Cartridge"
- board text removed: "EDGEBERRY"
- board text removed: "REV.: 1.5, Mid 2024"
